File: Experimental/PhatStats Experimental PCB/Resources/ESP32/LOLIN D32/PhatStats Slim Enclosure ESP Lolin D32 XTP2046 PCB v1.0 .sch (EAGLE design)
At the start: 32 parts, among them J3 455-1750-1-ND, Q1-PWM BC817-16LT1SMD, U3 XPT2046

Commit message: update
Parts:
- removed C2, C3, C4: 0.1uf, rcl:C-EUC1206
- removed J3: 455-1750-1-ND, SparkFun-Connectors:CONN_03
- removed NEO3, NEO4: WS2812B5050, adafruit:WS2812B5050
- removed Q1-PWM: BC817-16LT1SMD, transistor-npn:BC817-16LT1SMD
- removed R5: 10k, resistor:R-US_M1206
- removed R6: 10r, resistor:R-US_M1206
- removed SJ1: (no value), jumper:SJ2W
- removed SJ2, SJ3: (no value), jumper:SJ
- removed U$9: SMD_HEADERS_3PIN, TML_SMD_Headers_2.54_NoDrill:SMD_HEADERS_3PIN
- removed U1: (no value), TML_Seeeduino XIAO_QTPY_ThroughHole_ONLY_V1.1:MOUDLE-SEEEDUINO-XIAO
- added BAT: (no value), jst-ph:JST-PH2
- added BATT: S2B-PH-SM4-TB, con-JST PH:S2B-PH-SM4-TB
- added BLR5: 10r, resistor:R-US_M1206
- added BMS: DW01BATTERYPROT, TML_DW01_BatteryProtectionModule2:DW01BATTERYPROT
- added J4: (no value), SparkFun-Connectors:CONN_05
- added Q1_BL: BC817-16LT1SMD, transistor-npn:BC817-16LT1SMD
- added R3, R9: 10k, resistor:R-US_M1206
- added R8: 1k, resistor:R-US_M1206
- added S3: MOMENTARY-SWITCH-SPST-SMD-6.2MM-TALL, SparkFun-Switches:MOMENTARY-SWITCH-SPST-SMD-6.2MM-TALL
- added U$1: SMD_HEADERS_16PIN_2.54_NODRILLSSMD_HEADERS_16PIN, TML_SMD_Headers_2.54_NoDrill:SMD_HEADERS_16PIN_2.54_NODRILLSSMD_HEADERS_16PIN
- added U$11: SMD_HEADERS_5PIN_2.54_NODRILLS, TML_SMD_Headers_2.54_NoDrill:SMD_HEADERS_5PIN_2.54_NODRILLS
- J2: device SparkFun-Connectors:CONN_05 -> SparkFun-Connectors:CONN_04PTH
- R4: value 1k -> 10k
- S1: value MOMENTARY-SWITCH-SPST-SMD-6.2MM-TALL -> MOMENTARY-SWITCH-SPST-PTH-6.0MM; device SparkFun-Switches:MOMENTARY-SWITCH-SPST-SMD-6.2MM-TALL -> SparkFun-Switches:MOMENTARY-SWITCH-SPST-PTH-6.0MM
- S2: value MOMENTARY-SWITCH-SPST-SMD-6.2MM-TALL -> SK-12F14(1P2T)0.5A50VDC3MMPITCH; device SparkFun-Switches:MOMENTARY-SWITCH-SPST-SMD-6.2MM-TALL -> TML_SK-12F14(1P2T) 90D 0.5a 50vdc 3mm pitch:SK-12F14(1P2T)0.5A50VDC3MMPITCH
- U$2: value SMD_HEADERS_5PIN_2.54_NODRILLS -> TML_LOLIND32; device TML_SMD_Headers_2.54_NoDrill:SMD_HEADERS_5PIN_2.54_NODRILLS -> TML_Wemos Lolin D32 ESP32 Round Corrected:TML_LOLIND32
- U$4: value SMD_HEADERS_7PIN_2.54_NODRILLS -> SMD_HEADERS_16PIN_2.54_NODRILLSSMD_HEADERS_16PIN; device TML_SMD_Headers_2.54_NoDrill:SMD_HEADERS_7PIN_2.54_NODRILLS -> TML_SMD_Headers_2.54_NoDrill:SMD_HEADERS_16PIN_2.54_NODRILLSSMD_HEADERS_16PIN
- U$7: value SMD_HEADERS_7PIN_2.54_NODRILLS -> SMD_HEADERS_4PIN; device TML_SMD_Headers_2.54_NoDrill:SMD_HEADERS_7PIN_2.54_NODRILLS -> TML_SMD_Headers_2.54_NoDrill:SMD_HEADERS_4PIN
Connections:
- net NEODATA renamed N$2
- removed net BACKLIGHT_SDA: 0.LEDA, R4.2, U$3.BL, U$4.5, U$5.BL, U1.PA8_A4_D4_SDA
- removed net CS_SCL: 0.CSX, U$3.CS, U$4.6, U$5.CS, U1.PA9_A5_D5_SCL
- removed net N$2 (its old number): Q1-PWM.B, R4.1, R5.1
- removed net N$3: NEO2.DO, NEO3.DI
- removed net N$5: NEO3.DO, NEO4.DI
- removed net N$6: Q1-PWM.C, R6.1
- removed net NEO_OUT: J3.3, NEO4.DO, U$9.3
- new net BACKLIGHT: 0.LEDA, R8.2, U$2.GPIO4, U$3.BL, U$4.12, U$5.BL
- new net BATT+: BAT.2, BATT.1, BMS.P$4, R3.2
- new net BATT-: BAT.1, BATT.2, S2.P
- new net BATTMON: R3.1, R4.2, U$1.5, U$2.GPIO34
- new net BATTVCC: BMS.P$3, U$1.16, U$2.BAT
- new net BL: BLR5.1, Q1_BL.C
- new net CS: 0.CSX, U$2.GPIO17, U$3.CS, U$4.10, U$5.CS
- new net IR: U$1.13, U$2.GPIO13
- new net N$7: Q1_BL.B, R8.1, R9.1
- new net SCL: J2.3, U$2.GPIO22/SCL, U$4.3, U$7.3
- new net SDA: J2.4, U$2.GPIO21/SDA, U$4.6, U$7.4
- net BLGND: now also BLR5.2; no longer R6.2
- net DC: now also U$2.GPIO16, U$4.11; no longer U$7.7, U1.PB09_A7_D7_RX
- net ENC_A: now also J4.4, U$1.11, U$11.4, U$2.GPIO14; no longer J2.4, SJ3.1, U$2.4, U$4.4, U1.PA11_A3_D3
- net ENC_B: now also J4.5, U$1.10, U$11.5, U$2.GPIO27; no longer J2.5, SJ2.1, U$2.5, U$4.3, U1.PA10_A2_D2
- net ENC_BUTTON: now also J4.3, S3.2, U$11.3, U$2.GPIO0, U$4.13; no longer J2.3, SJ1.1, U$2.3, U$4.2, U1.PA4_A1_D1
- net GND: now also BMS.P$2, J4.1, Q1_BL.E, R4.1, S3.1, U$11.1, U$2.GND, U$4.1, U$4.16, U$7.1; no longer C2.2, C3.2, C4.2, J3.2, NEO3.GND, NEO4.GND, Q1-PWM.E, S2.1, U$2.1, U$7.2, U$9.2, U1.GND
- net MISO: now also U$2.MI/GPIO19, U$4.7; no longer U$7.5, U1.PA5_A9_D9_MISO
- net MOSI: now also U$2.MO/GPIO23, U$4.2; no longer SJ1.3, U$7.4, U1.PA6_A10_D10_MOSI
- net N$1: now also BMS.P$1, S2.O; no longer S2.2, SJ1.2
- net NEO: now also U$2.GPIO2, U$4.14; no longer U$4.7, U1.PB08_A6_D6_TX
- net RST: now also U$2.GPIO15, U$4.15; no longer U$4.1, U1.PA02_A0_D0
- net SCK: now also U$2.SCK/GPIO18, U$4.8; no longer U$7.6, U1.PA7_A8_D8_SCK
- net T_CS: now also U$1.7, U$2.GPIO33; no longer SJ2.2
- net T_IRQ: now also U$1.6, U$2.GPIO32; no longer SJ3.2
- net VCC: now also J4.2, R9.2, U$1.1, U$11.2, U$2.3V3, U$7.2; no longer C2.1, C3.1, C4.1, J3.1, NEO3.VDD, NEO4.VDD, R5.2, U$2.2, U$7.3, U$9.1, U1.3V3
Other:
- note added: "2.8" ILI9341 TFT"
- note added: "Battery Managment"
- note added: "Battery Protection Module DW01"
- note added: "ESP32"
- note added: "Infra Red"
- note added: "MCU Battery Level Monitor (ADC)"
- note added: "Neo Pixels"
- note added: "PWM Backlight"
- note added: "SMD BMS OUT PH2"
- note added: "SMD Battery PH2 Connector"
- note added: "https://www.wemos.cc/en/latest/d32/d32.html#documentation"
- note added: "i2C / SPi Accessory Headers"
- note removed: "Button (s2) option Jumper"
- note removed: "NeoPixels"
- note removed: "Rotary Encoder"
- note removed: "TFT Bare Screen PWM"
- moved on the sheet: C1, CT1, CT2, R2, R4, RT1, S1, U3
