File: Experimental/PhatStats Experimental PCB/Resources/QTPY/PhatStats Slim Enclosure QTPY PCB v1.00 RTM XPT2406 .sch (EAGLE design)
At the start: 33 parts, among them J1 1X2-3.5MM, Q1_BL BC817-16LT1SMD, U3 XPT2046

Commit message: update
Parts:
- removed BAT: (no value), jst-ph:JST-PH2
- removed BATT: S2B-PH-SM4-TB, con-JST PH:S2B-PH-SM4-TB
- removed BLR5: 10r, resistor:R-US_M1206
- removed DW01-BMS: DW01BATTERYPROT, TML_DW01_BatteryProtectionModule2:DW01BATTERYPROT
- removed J1: 1X2-3.5MM, adafruit:1X2-3.5MM
- removed J4: (no value), SparkFun-Connectors:CONN_05
- removed PAD1, PAD2: WIREPADSMD5-1,8, wirepad:WIREPADSMD5-1,8
- removed Q1_BL: BC817-16LT1SMD, transistor-npn:BC817-16LT1SMD
- removed R3, R9: 10k, resistor:R-US_M1206
- removed R8: 1k, resistor:R-US_M1206
- removed S3: MOMENTARY-SWITCH-SPST-SMD-6.2MM-TALL, SparkFun-Switches:MOMENTARY-SWITCH-SPST-SMD-6.2MM-TALL
- removed U$1: SMD_HEADERS_13PIN_2.54_NODRILLS, TML_SMD_Headers_2.54_NoDrill:SMD_HEADERS_13PIN_2.54_NODRILLS
- removed U$11: SMD_HEADERS_5PIN_2.54_NODRILLS, TML_SMD_Headers_2.54_NoDrill:SMD_HEADERS_5PIN_2.54_NODRILLS
- removed U$8: SMD_HEADERS_4PIN, TML_SMD_Headers_2.54_NoDrill:SMD_HEADERS_4PIN
- added C2, C3, C4: 0.1uf, rcl:C-EUC1206
- added J3: 455-1750-1-ND, SparkFun-Connectors:CONN_03
- added NEO3, NEO4: WS2812B5050, adafruit:WS2812B5050
- added Q1-PWM: BC817-16LT1SMD, transistor-npn:BC817-16LT1SMD
- added R5: 10k, resistor:R-US_M1206
- added R6: 10r, resistor:R-US_M1206
- added SJ1: (no value), jumper:SJ2W
- added SJ2, SJ3: (no value), jumper:SJ
- added U$4: SMD_HEADERS_7PIN_2.54_NODRILLS, TML_SMD_Headers_2.54_NoDrill:SMD_HEADERS_7PIN_2.54_NODRILLS
- added U$9: SMD_HEADERS_3PIN, TML_SMD_Headers_2.54_NoDrill:SMD_HEADERS_3PIN
- added U1: (no value), TML_Seeeduino XIAO_QTPY_ThroughHole_ONLY_V1.1:MOUDLE-SEEEDUINO-XIAO
- J2: device SparkFun-Connectors:CONN_04PTH -> SparkFun-Connectors:CONN_05
- R4: value 10k -> 1k
- S1: value MOMENTARY-SWITCH-SPST-PTH-6.0MM -> MOMENTARY-SWITCH-SPST-SMD-6.2MM-TALL; device SparkFun-Switches:MOMENTARY-SWITCH-SPST-PTH-6.0MM -> SparkFun-Switches:MOMENTARY-SWITCH-SPST-SMD-6.2MM-TALL
- S2: value SK-12F14(1P2T)0.5A50VDC3MMPITCH -> MOMENTARY-SWITCH-SPST-SMD-6.2MM-TALL; device TML_SK-12F14(1P2T) 90D 0.5a 50vdc 3mm pitch:SK-12F14(1P2T)0.5A50VDC3MMPITCH -> SparkFun-Switches:MOMENTARY-SWITCH-SPST-SMD-6.2MM-TALL
- U$2: value SMD_HEADERS_13PIN_2.54_NODRILLS -> SMD_HEADERS_5PIN_2.54_NODRILLS; device TML_SMD_Headers_2.54_NoDrill:SMD_HEADERS_13PIN_2.54_NODRILLS -> TML_SMD_Headers_2.54_NoDrill:SMD_HEADERS_5PIN_2.54_NODRILLS
- U$7: value (none) -> SMD_HEADERS_7PIN_2.54_NODRILLS; device TML_Wemos LOLIN32 LITE ESP32 Round Pads:TML_LOLIND32_LITE -> TML_SMD_Headers_2.54_NoDrill:SMD_HEADERS_7PIN_2.54_NODRILLS
Connections:
- net N$2 renamed NEODATA
- removed net BACKLIGHT: 0.LEDA, R8.2, U$2.9, U$3.BL, U$5.BL, U$7.4
- removed net BATT+: BAT.2, BATT.1, DW01-BMS.P$4, R3.2
- removed net BATT-: BAT.1, BATT.2, S2.P
- removed net BATTMON: R3.1, R4.2, U$1.4, U$7.34
- removed net BATTVCC: DW01-BMS.P$3, J1.1, PAD2.P
- removed net BL: BLR5.1, Q1_BL.C
- removed net CS: 0.CSX, U$2.7, U$3.CS, U$5.CS, U$7.17
- removed net IR: U$2.13, U$7.13
- removed net MISO_SDA: 0.SDO, J2.4, U$2.3, U$3.MISO, U$3.T_DO, U$5.MISO, U$5.T_DO, U$7.19, U$8.4, U3.DOUT
- removed net MOSI_SCL: 0.SDI, J2.3, U$2.4, U$3.MOSI, U$3.T_DIN, U$5.MOSI, U$5.T_DIN, U$7.23, U$8.3, U3.DIN
- removed net N$7: Q1_BL.B, R8.1, R9.1
- new net BACKLIGHT_SDA: 0.LEDA, R4.2, U$3.BL, U$4.5, U$5.BL, U1.PA8_A4_D4_SDA
- new net CS_SCL: 0.CSX, U$3.CS, U$4.6, U$5.CS, U1.PA9_A5_D5_SCL
- new net MISO: 0.SDO, U$3.MISO, U$3.T_DO, U$5.MISO, U$5.T_DO, U$7.5, U1.PA5_A9_D9_MISO, U3.DOUT
- new net MOSI: 0.SDI, SJ1.3, U$3.MOSI, U$3.T_DIN, U$5.MOSI, U$5.T_DIN, U$7.4, U1.PA6_A10_D10_MOSI, U3.DIN
- new net N$2: Q1-PWM.B, R4.1, R5.1
- new net N$3: NEO2.DO, NEO3.DI
- new net N$5: NEO3.DO, NEO4.DI
- new net N$6: Q1-PWM.C, R6.1
- new net NEO_OUT: J3.3, NEO4.DO, U$9.3
- net BLGND: now also R6.2; no longer BLR5.2
- net DC: now also U$7.7, U1.PB09_A7_D7_RX; no longer U$2.8, U$7.16
- net ENC_A: now also J2.4, SJ3.1, U$2.4, U$4.4, U1.PA11_A3_D3; no longer J4.4, U$1.11, U$11.4, U$7.14
- net ENC_B: now also J2.5, SJ2.1, U$2.5, U$4.3, U1.PA10_A2_D2; no longer J4.5, U$1.10, U$11.5, U$7.27
- net ENC_BUTTON: now also J2.3, SJ1.1, U$2.3, U$4.2, U1.PA4_A1_D1; no longer J4.3, S3.2, U$11.3, U$2.10, U$7.0
- net GND: now also C2.2, C3.2, C4.2, J3.2, NEO3.GND, NEO4.GND, Q1-PWM.E, S2.1, U$2.1, U$7.2, U$9.2, U1.GND; no longer DW01-BMS.P$2, J1.2, J4.1, PAD1.P, Q1_BL.E, R4.1, S3.1, U$1.13, U$11.1, U$7.GND, U$8.1
- net N$1: now also S2.2, SJ1.2; no longer DW01-BMS.P$1, S2.O
- net NEO: now also U$4.7, U1.PB08_A6_D6_TX; no longer U$2.11, U$7.2
- net RST: now also U$4.1, U1.PA02_A0_D0; no longer U$2.12, U$7.15
- net SCK: now also U$7.6, U1.PA7_A8_D8_SCK; no longer U$2.5, U$7.18
- net T_CS: now also SJ2.2; no longer U$1.7, U$7.33
- net T_IRQ: now also SJ3.2; no longer U$1.6, U$7.32
- net VCC: now also C2.1, C3.1, C4.1, J3.1, NEO3.VDD, NEO4.VDD, R5.2, U$2.2, U$7.3, U$9.1, U1.3V3; no longer J4.2, R9.2, U$11.2, U$2.1, U$7.3V, U$8.2
Other:
- note added: "Button (s2) option Jumper"
- note added: "NeoPixels"
- note added: "Rotary Encoder"
- note added: "TFT Bare Screen PWM"
- note removed: "2.8" ILI9341 TFT"
- note removed: "Battery Managment"
- note removed: "Battery Protection Module DW01"
- note removed: "CHECK BL RESISTOR!!!"
- note removed: "ESP32"
- note removed: "Fix Grounding Sort Switch"
- note removed: "Infra Red"
- note removed: "MCU Battery Level Monitor (ADC)"
- note removed: "Neo Pixels"
- note removed: "PWM Backlight"
- note removed: "SMD BMS OUT PH2"
- note removed: "SMD Battery PH2 Connector"
- note removed: "https://www.wemos.cc/en/latest/d32/d32.html#documentation"
- note removed: "i2C / SPi Accessory Headers"
- moved on the sheet: C1, CT1, CT2, R2, R4, RT1, S1, U3
