File: Experimental/PhatStats Experimental PCB/Resources/QTPY/PhatStats Slim Enclosure 2.8 ILI9341 QTPY XIAO PCB v1.0c XPT2406 .sch (EAGLE design)
At the start: 32 parts, among them J3 455-1750-1-ND, Q1-PWM BC817-16LT1SMD, U3 XPT2046

Commit message: update
Parts:
- removed NEO4: WS2812B5050, adafruit:WS2812B5050
- added NEO0: WS2812B5050, adafruit:WS2812B5050
- R4: value 1k -> 1 to 10k
- U$3: device TML_ili9341-2.8_tft-display_Corrected:2.8_TFT -> TML_ili9341-2.8_tft-display_Corrected v2:2.8_TFT
Connections:
- removed net N$5 (its old number): NEO3.DO, NEO4.DI
- new net N$3: NEO1.DO, NEO2.DI
- net GND: now also NEO0.GND; no longer NEO4.GND
- net N$4: now also NEO0.DI; no longer NEO1.DI
- net NEODATA: now also NEO0.DO, NEO1.DI; no longer NEO1.DO, NEO2.DI
- net NEO_OUT: now also NEO3.DO; no longer NEO4.DO
- net VCC: now also NEO0.VDD; no longer NEO4.VDD
Other:
- note added: "Optional"
- note added: "S8050 J3Y NPN SOT-23 SMD 0.5A 25v"
- moved on the sheet: CT1, CT2, R5, RT1, S2, SJ1, U3
