File: Experimental/PhatStats Experimental PCB/Resources/ESP32/LOLIN32 LITE/PhatStats Slim Enclosure ESP Lolin32 LITE XTP2046 PCB v1c Corrected.sch (EAGLE design)
At the start: 30 parts, among them Q1_BL BC817-16LT1SMD, U3 XPT2046

Commit message: update
Parts:
- removed NEO2: WS2812B5050, adafruit:WS2812B5050
- removed U$4: SMD_HEADERS_16PIN_2.54_NODRILLSSMD_HEADERS_16PIN, TML_SMD_Headers_2.54_NoDrill:SMD_HEADERS_16PIN_2.54_NODRILLSSMD_HEADERS_16PIN
- added J1: 1X2-3.5MM, adafruit:1X2-3.5MM
- added NEO0: WS2812B5050, adafruit:WS2812B5050
- added PAD1, PAD2: WIREPADSMD5-1,8, wirepad:WIREPADSMD5-1,8
- added U$8: SMD_HEADERS_4PIN, TML_SMD_Headers_2.54_NoDrill:SMD_HEADERS_4PIN
- R8: value 1k -> 1 to 10k
- S2: device TML_SK-12F14(1P2T) 90D 0.5a 50vdc 3mm pitch:SK-12F14(1P2T)0.5A50VDC3MMPITCH -> TML_SK-12F14(1P2T) 90Deg 0.5a 50vdc 3mm pitch Round Pads:SK-12F14(1P2T)0.5A50VDC3MMPITCH
- U$1: value SMD_HEADERS_16PIN_2.54_NODRILLSSMD_HEADERS_16PIN -> SMD_HEADERS_13PIN_2.54_NODRILLS; device TML_SMD_Headers_2.54_NoDrill:SMD_HEADERS_16PIN_2.54_NODRILLSSMD_HEADERS_16PIN -> TML_SMD_Headers_2.54_NoDrill:SMD_HEADERS_13PIN_2.54_NODRILLS
- U$2: value TML_LOLIND32 -> SMD_HEADERS_13PIN_2.54_NODRILLS; device TML_Wemos Lolin D32 ESP32 Round Corrected:TML_LOLIND32 -> TML_SMD_Headers_2.54_NoDrill:SMD_HEADERS_13PIN_2.54_NODRILLS
- U$3: device TML_ili9341-2.8_tft-display_Corrected:2.8_TFT -> TML_ili9341-2.8_tft-display_Corrected v2:2.8_TFT
- U$7: value SMD_HEADERS_4PIN -> (none); device TML_SMD_Headers_2.54_NoDrill:SMD_HEADERS_4PIN -> TML_Wemos LOLIN32 LITE ESP32 Round Pads:TML_LOLIND32_LITE
- renumbered BMS to DW01-BMS
Connections:
- removed net MISO: 0.SDO, U$2.MI/GPIO19, U$3.MISO, U$3.T_DO, U$4.7, U$5.MISO, U$5.T_DO, U3.DOUT
- removed net MOSI: 0.SDI, U$2.MO/GPIO23, U$3.MOSI, U$3.T_DIN, U$4.2, U$5.MOSI, U$5.T_DIN, U3.DIN
- removed net SCL: J2.3, U$2.GPIO22/SCL, U$4.3, U$7.3
- removed net SDA: J2.4, U$2.GPIO21/SDA, U$4.6, U$7.4
- new net MISO_SDA: 0.SDO, J2.4, U$2.3, U$3.MISO, U$3.T_DO, U$5.MISO, U$5.T_DO, U$7.19, U$8.4, U3.DOUT
- new net MOSI_SCL: 0.SDI, J2.3, U$2.4, U$3.MOSI, U$3.T_DIN, U$5.MOSI, U$5.T_DIN, U$7.23, U$8.3, U3.DIN
- net BACKLIGHT: now also U$2.9, U$7.4; no longer U$2.GPIO4, U$4.12
- net BATTMON: now also U$1.4, U$7.34; no longer U$1.5, U$2.GPIO34
- net BATTVCC: now also J1.1, PAD2.P; no longer U$1.16, U$2.BAT
- net CS: now also U$2.7, U$7.17; no longer U$2.GPIO17, U$4.10
- net DC: now also U$2.8, U$7.16; no longer U$2.GPIO16, U$4.11
- net ENC_A: now also U$7.14; no longer U$2.GPIO14
- net ENC_B: now also U$7.27; no longer U$2.GPIO27
- net ENC_BUTTON: now also U$2.10, U$7.0; no longer U$2.GPIO0, U$4.13
- net GND: now also J1.2, NEO0.GND, PAD1.P, U$1.13, U$7.GND, U$8.1; no longer NEO2.GND, U$2.GND, U$4.1, U$4.16, U$7.1
- net IR: now also U$2.13, U$7.13; no longer U$1.13, U$2.GPIO13
- net N$2: now also NEO0.DO, NEO1.DI; no longer NEO1.DO, NEO2.DI
- net N$4: now also NEO0.DI; no longer NEO1.DI
- net NEO: now also U$2.11, U$7.2; no longer U$2.GPIO2, U$4.14
- net RST: now also U$2.12, U$7.15; no longer U$2.GPIO15, U$4.15
- net SCK: now also U$2.5, U$7.18; no longer U$2.SCK/GPIO18, U$4.8
- net T_CS: now also U$7.33; no longer U$2.GPIO33
- net T_IRQ: now also U$7.32; no longer U$2.GPIO32
- net VCC: now also NEO0.VDD, U$2.1, U$7.3V, U$8.2; no longer NEO2.VDD, U$1.1, U$2.3V3, U$7.2
Other:
- note added: "Optional"
- note added: "S8050 J3Y NPN SOT-23 SMD 0.5A 25v"
- moved on the sheet: BLR5, CT1, CT2, J2, J4, Q1_BL, R8, R9, RT1, U$11, U3
